File: PCB/sensores.kicad_pcb (KiCad board)
At the start: 2 copper layers, 80.6 x 50 mm, 7 parts, among them P10 CONN_01X07, P11 CONN_01X07, P15 DHT22, P16 GY-87, P2 CONN_01X04, P3 CONN_01X04

Commit message: Fix PCBs
Changed lines of the file:
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@@
-(kicad_pcb (version 4) (host pcbnew 4.0.0-rc1-stable)
+(kicad_pcb (version 4) (host pcbnew 4.0.2+dfsg1-stable)
   (general
     (links 11)
@@
   )
   (layers
-    (0 F.Cu signal)
-    (31 B.Cu signal)
+    (0 F.Cu signal hide)
+    (31 B.Cu signal hide)
     (32 B.Adhes user)
     (33 F.Adhes user)
@@
     (descr "Through hole pin header")
     (tags "pin header")
-    (fp_text reference P3 (at 0 -5.1 270) (layer F.SilkS)
+    (fp_text reference P3 (at 0.25 -2.73 270) (layer F.SilkS)
       (effects (font (size 1 1) (thickness 0.15)))
     )
@@
     (descr "Through hole pin header")
     (tags "pin header")
-    (fp_text reference P10 (at 0 -5.1) (layer F.SilkS)
+    (fp_text reference P10 (at 3.45 -0.25) (layer F.SilkS)
       (effects (font (size 1 1) (thickness 0.15)))
     )
@@
     (descr "Through hole pin header")
     (tags "pin header")
-    (fp_text reference P11 (at 0 -5.1 90) (layer F.SilkS)
+    (fp_text reference P11 (at 0 -2.95 90) (layer F.SilkS)
       (effects (font (size 1 1) (thickness 0.15)))
     )
@@
     (descr "Through hole pin header")
     (tags "pin header")
-    (fp_text reference P15 (at 0 -5.1 270) (layer F.SilkS)
-      (effects (font (size 1 1) (thickness 0.15)))
-    )
-    (fp_text value DHT22 (at 0 -3.1 270) (layer F.Fab)
+    (fp_text reference P15 (at 0.2 -2.8 270) (layer F.SilkS)
+      (effects (font (size 1 1) (thickness 0.15)))
+    )
+    (fp_text value DHT22 (at 3.4 1.8 360) (layer F.SilkS)
       (effects (font (size 1 1) (thickness 0.15)))
     )
@@
     (descr "Through hole pin header")
     (tags "pin header")
-    (fp_text reference P16 (at 0 -5.1 180) (layer F.SilkS)
-      (effects (font (size 1 1) (thickness 0.15)))
-    )
-    (fp_text value GY-87 (at 0 -3.1 180) (layer F.Fab)
+    (fp_text reference P16 (at 0 -3.34 180) (layer F.SilkS)
+      (effects (font (size 1 1) (thickness 0.15)))
+    )
+    (fp_text value GY-87 (at 2.65 9.86 270) (layer F.SilkS)
       (effects (font (size 1 1) (thickness 0.15)))
     )
@@
     (descr "Through hole pin header")
     (tags "pin header")
-    (fp_text reference P2 (at 0 -5.1) (layer F.SilkS)
-      (effects (font (size 1 1) (thickness 0.15)))
-    )
+    (fp_text reference P2 (at 0.25 -2.75) (layer F.SilkS)
+      (effects (font (size 1 1) (thickness 0.15)))
+    )
