File: Telemetrysch.sch (KiCad schematic (older format))
At the start: 2 parts

Commit message: Schematic v0.2
Added IC and wiring
Parts:
- removed MODULE?: L80-M39, QUECTEL_L80-M39, symbol L80-M39
- removed U?: RFM95W-868S2, XCVR_RFM95W-868S2, symbol RFM95W-868S2
- added MODULE1: L80-M39, QUECTEL_L80-M39, symbol L80-M39
- added P10, P7: CONN_01X07, symbol CONN_01X07
- added P6: ANT, symbol CONN_01X01
- added P8, P9: CONN_01X04, symbol CONN_01X04
- added U2: RFM95W-868S2, XCVR_RFM95W-868S2, symbol RFM95W-868S2
Connections:
- net labels added: +BATT, A0, A1, A2, A3, D7, D8, DHT/D6, GND, INT0, INT1, MISO, MOSI, NSS, RST, SCK, SCL, SDA, S_RX, S_TX
- wire segments 0 -> 74
- no-connect marks 0 -> 11

Commit message: Fix arduino mini pro pin 6 bug, added capacitors
Parts:
- removed P6: ANT, symbol CONN_01X01
- added A1: ANT, LoRa:SMA_Conn_Ant, symbol ANT
- added C3: C, symbol C
- MODULE1: footprint QUECTEL_L80-M39 -> CatSat:L80
- P10, P7: footprint (none) -> Pin_Headers:Pin_Header_Straight_1x07
- P8, P9: footprint (none) -> Pin_Headers:Pin_Header_Straight_1x04
- U2: footprint XCVR_RFM95W-868S2 -> LoRa:RFM
Connections:
- wire segments 74 -> 81

Commit message: Finished telemtry PCB
Parts:
- C3: footprint (none) -> Capacitors_ThroughHole:C_Disc_D6_P5
Changed lines of the file:
@@
 $EndComp
 $Comp
-L +BATT #PWR09
+L +BATT #PWR011
 U 1 1 5799299F
 P 5325 2435
-F 0 "#PWR09" H 5325 2285 50  0001 C CNN
+F 0 "#PWR011" H 5325 2285 50  0001 C CNN
 F 1 "+BATT" H 5325 2575 50  0000 C CNN
 F 2 "" H 5325 2435 50  0000 C CNN
@@
 A0
 $Comp
-L GND #PWR010
+L GND #PWR012
 U 1 1 579929AE
 P 5020 1980
-F 0 "#PWR010" H 5020 1730 50  0001 C CNN
+F 0 "#PWR012" H 5020 1730 50  0001 C CNN
 F 1 "GND" H 5020 1830 50  0000 C CNN
 F 2 "" H 5020 1980 50  0000 C CNN
@@
 NoConn ~ 3990 4105
 $Comp
-L GND #PWR011
+L GND #PWR013
 U 1 1 57994B3D
 P 5990 4195
-F 0 "#PWR011" H 5990 3945 50  0001 C CNN
+F 0 "#PWR013" H 5990 3945 50  0001 C CNN
 F 1 "GND" H 5990 4045 50  0000 C CNN
 F 2 "" H 5990 4195 50  0000 C CNN
@@
 MOSI
 $Comp
-L +BATT #PWR012
+L +BATT #PWR014
 U 1 1 57994EF9
 P 5800 3095
-F 0 "#PWR012" H 5800 2945 50  0001 C CNN
+F 0 "#PWR014" H 5800 2945 50  0001 C CNN
 F 1 "+BATT" H 5800 3235 50  0000 C CNN
 F 2 "" H 5800 3095 50  0000 C CNN
@@
 $EndComp
 $Comp
-L GND #PWR013
+L GND #PWR015
 U 1 1 57995F4A
 P 8935 4365
-F 0 "#PWR013" H 8935 4115 50  0001 C CNN
+F 0 "#PWR015" H 8935 4115 50  0001 C CNN
 F 1 "GND" H 8935 4215 50  0000 C CNN
 F 2 "" H 8935 4365 50  0000 C CNN
@@
 NoConn ~ 8910 3135
 $Comp
-L +BATT #PWR014
+L +BATT #PWR016
 U 1 1 57996632
 P 8910 2905
-F 0 "#PWR014" H 8910 2755 50  0001 C CNN
+F 0 "#PWR016" H 8910 2755 50  0001 C CNN
 F 1 "+BATT" H 8910 3045 50  0000 C CNN
 F 2 "" H 8910 2905 50  0000 C CNN
@@
 D7
 $Comp
-L +BATT #PWR015
+L +BATT #PWR017
 U 1 1 579A7853
 P 9335 4005
-F 0 "#PWR015" H 9335 3855 50  0001 C CNN
+F 0 "#PWR017" H 9335 3855 50  0001 C CNN
 F 1 "+BATT" H 9335 4145 50  0000 C CNN
 F 2 "" H 9335 4005 50  0000 C CNN
@@
 $EndComp
 $Comp
-L GND #PWR016
+L GND #PWR018
 U 1 1 579A787C
 P 9300 4305
-F 0 "#PWR016" H 9300 4055 50  0001 C CNN
+F 0 "#PWR018" H 9300 4055 50  0001 C CNN
 F 1 "GND" H 9300 4155 50  0000 C CNN
 F 2 "" H 9300 4305 50  0000 C CNN
@@
 $EndComp
 $Comp
-L GND #PWR017
+L GND #PWR019
 U 1 1 57994571
 P 6165 3815
-F 0 "#PWR017" H 6165 3815 30  0001 C CNN
+F 0 "#PWR019" H 6165 3815 30  0001 C CNN
 F 1 "GND" H 6165 3745 30  0001 C CNN
 F 2 "" H 6165 3815 60  0000 C CNN
@@
 $EndComp
 $Comp
-L GND #PWR018
-U 1 1 57994593
-P 6315 3815
-F 0 "#PWR018" H 6315 3815 30  0001 C CNN
-F 1 "GND" H 6315 3745 30  0001 C CNN
-F 2 "" H 6315 3815 60  0000 C CNN
-F 3 "" H 6315 3815 60  0000 C CNN
-	1    6315 3815
-	1    0    0    -1
-$EndComp
-$Comp
-L GND #PWR019
-U 1 1 5799467C
-P 6160 2985
-F 0 "#PWR019" H 6160 2985 30  0001 C CNN
-F 1 "GND" H 6160 2915 30  0001 C CNN
-F 2 "" H 6160 2985 60  0000 C CNN
-F 3 "" H 6160 2985 60  0000 C CNN
-	1    6160 2985
+L GND #PWR022
+U 1 1 5799469E
+P 6165 3055
+F 0 "#PWR022" H 6165 3055 30  0001 C CNN
+F 1 "GND" H 6165 2985 30  0001 C CNN
+F 2 "" H 6165 3055 60  0000 C CNN
+F 3 "" H 6165 3055 60  0000 C CNN
+	1    6165 3055
 	-1   0    0    1
 $EndComp
-$Comp
-L GND #PWR020
-U 1 1 5799469E
-P 6315 2990
-F 0 "#PWR020" H 6315 2990 30  0001 C CNN
-F 1 "GND" H 6315 2920 30  0001 C CNN
-F 2 "" H 6315 2990 60  0000 C CNN
-F 3 "" H 6315 2990 60  0000 C CNN
-	1    6315 2990
-	-1   0    0    1
-$EndComp
-Wire Wire Line
-	6315 3055 6315 2990
-Wire Wire Line
-	6160 2985 6160 3055
-Wire Wire Line
-	6160 3055 6165 3055
 Wire Wire Line
 	6165 3815 6165 3755
@@
 F 0 "C3" H 8275 1795 50  0000 L CNN
 F 1 "C" H 8275 1595 50  0000 L CNN
-F 2 "" H 8288 1545 30  0000 C CNN
+F 2 "Capacitors_ThroughHole:C_Disc_D6_P5" H 8288 1545 30  0001 C CNN
 F 3 "" H 8250 1695 60  0000 C CNN
 	1    8250 1695
@@
 $EndComp
 $Comp
-L GND #PWR?
+L GND #PWR023
 U 1 1 579BD6A9
 P 8250 1910
-F 0 "#PWR?" H 8250 1910 30  0001 C CNN
+F 0 "#PWR023" H 8250 1910 30  0001 C CNN
 F 1 "GND" H 8250 1840 30  0001 C CNN
 F 2 "" H 8250 1910 60  0000 C CNN
@@
 	8250 1910 8250 1845
 $Comp
-L +BATT #PWR?
+L +BATT #PWR024
 U 1 1 579BDAA7
 P 8250 1500
-F 0 "#PWR?" H 8250 1350 50  0001 C CNN
+F 0 "#PWR024" H 8250 1350 50  0001 C CNN
 F 1 "+BATT" H 8250 1640 50  0000 C CNN
 F 2 "" H 8250 1500 50  0000 C CNN
@@
 Wire Wire Line
 	8250 1500 8250 1545
+$Comp
+L GND #PWR?
+U 1 1 579F7DD8
+P 6315 3055
+F 0 "#PWR?" H 6315 3055 30  0001 C CNN
+F 1 "GND" H 6315 2985 30  0001 C CNN
+F 2 "" H 6315 3055 60  0000 C CNN
+F 3 "" H 6315 3055 60  0000 C CNN
+	1    6315 3055
+	-1   0    0    1
+$EndComp
+$Comp
+L GND #PWR?
+U 1 1 579F7E1D
+P 6315 3815
+F 0 "#PWR?" H 6315 3815 30  0001 C CNN
+F 1 "GND" H 6315 3745 30  0001 C CNN
+F 2 "" H 6315 3815 60  0000 C CNN
+F 3 "" H 6315 3815 60  0000 C CNN
+	1    6315 3815
+	1    0    0    -1
+$EndComp
 $EndSCHEMATC

Commit message: PCB final
Parts:
- added R1, R2: R, Resistors_ThroughHole:Resistor_Horizontal_RM7mm, symbol R
Connections:
- net +BATT: now also MODULE1.5 (V_BCKP), R1.1, R2.1
- net NSS: now also R2.2
- net RST: now also R1.2
- no-connect marks 11 -> 10
Changed lines of the file:
@@
 NoConn ~ 8915 3635
 NoConn ~ 8915 3735
-NoConn ~ 8910 3135
 $Comp
 L +BATT #PWR016
@@
 	4175 3305 3995 3305
 Wire Wire Line
-	4175 3405 3995 3405
-Wire Wire Line
-	4175 3505 3985 3505
+	3705 3405 4175 3405
+Wire Wire Line
+	3385 3505 4175 3505
 Wire Wire Line
 	4175 3605 3985 3605
@@
 	8695 3035 8910 3035
 Wire Wire Line
-	8695 3135 8910 3135
+	8910 3135 8695 3135
 Wire Wire Line
 	8695 3535 8915 3535
@@
 	7495 3635 7325 3635
 Wire Wire Line
-	8910 3035 8910 2905
+	8910 2905 8910 3135
 Wire Wire Line
 	5230 1020 5230 1165
@@
 $EndComp
 $Comp
-L GND #PWR022
+L GND #PWR020
 U 1 1 5799469E
 P 6165 3055
-F 0 "#PWR022" H 6165 3055 30  0001 C CNN
+F 0 "#PWR020" H 6165 3055 30  0001 C CNN
 F 1 "GND" H 6165 2985 30  0001 C CNN
 F 2 "" H 6165 3055 60  0000 C CNN
@@
 $EndComp
 $Comp
-L GND #PWR023
+L GND #PWR021
 U 1 1 579BD6A9
 P 8250 1910
-F 0 "#PWR023" H 8250 1910 30  0001 C CNN
+F 0 "#PWR021" H 8250 1910 30  0001 C CNN
 F 1 "GND" H 8250 1840 30  0001 C CNN
 F 2 "" H 8250 1910 60  0000 C CNN
@@
 	8250 1910 8250 1845
 $Comp
-L +BATT #PWR024
+L +BATT #PWR022
 U 1 1 579BDAA7
 P 8250 1500
-F 0 "#PWR024" H 8250 1350 50  0001 C CNN
+F 0 "#PWR022" H 8250 1350 50  0001 C CNN
 F 1 "+BATT" H 8250 1640 50  0000 C CNN
 F 2 "" H 8250 1500 50  0000 C CNN
@@
 	8250 1500 8250 1545
 $Comp
-L GND #PWR?
+L GND #PWR023
 U 1 1 579F7DD8
 P 6315 3055
-F 0 "#PWR?" H 6315 3055 30  0001 C CNN
+F 0 "#PWR023" H 6315 3055 30  0001 C CNN
 F 1 "GND" H 6315 2985 30  0001 C CNN
 F 2 "" H 6315 3055 60  0000 C CNN
@@
 $EndComp
 $Comp
-L GND #PWR?
+L GND #PWR024
 U 1 1 579F7E1D
 P 6315 3815
-F 0 "#PWR?" H 6315 3815 30  0001 C CNN
+F 0 "#PWR024" H 6315 3815 30  0001 C CNN
 F 1 "GND" H 6315 3745 30  0001 C CNN
 F 2 "" H 6315 3815 60  0000 C CNN
@@
 	1    0    0    -1
 $EndComp
+Connection ~ 8910 3035
+$Comp
+L R R2
+U 1 1 579FEFF6
+P 3705 3205
+F 0 "R2" V 3785 3205 50  0000 C CNN
+F 1 "R" V 3705 3205 50  0000 C CNN
+F 2 "Resistors_ThroughHole:Resistor_Horizontal_RM7mm" V 3635 3205 30  0001 C CNN
+F 3 "" H 3705 3205 30  0000 C CNN
+	1    3705 3205
+	1    0    0    -1
+$EndComp
+$Comp
+L R R1
+U 1 1 579FF08B
+P 3385 3220
+F 0 "R1" V 3465 3220 50  0000 C CNN
+F 1 "R" V 3385 3220 50  0000 C CNN
+F 2 "Resistors_ThroughHole:Resistor_Horizontal_RM7mm" V 3315 3220 30  0001 C CNN
+F 3 "" H 3385 3220 30  0000 C CNN
+	1    3385 3220
+	1    0    0    -1
+$EndComp
+Wire Wire Line
+	3705 3355 3705 3405
+Wire Wire Line
+	3385 3505 3385 3370
+$Comp
+L +BATT #PWR025
+U 1 1 579FF70B
+P 3385 3070
+F 0 "#PWR025" H 3385 2920 50  0001 C CNN
+F 1 "+BATT" H 3385 3210 50  0000 C CNN
+F 2 "" H 3385 3070 50  0000 C CNN
+F 3 "" H 3385 3070 50  0000 C CNN
+	1    3385 3070
+	1    0    0    -1
+$EndComp
+$Comp
+L +BATT #PWR026
+U 1 1 579FF837
+P 3705 3055
+F 0 "#PWR026" H 3705 2905 50  0001 C CNN
+F 1 "+BATT" H 3705 3195 50  0000 C CNN
+F 2 "" H 3705 3055 50  0000 C CNN
+F 3 "" H 3705 3055 50  0000 C CNN
+	1    3705 3055
+	1    0    0    -1
+$EndComp
