File: PCB/earth_station/earth station.sch (KiCad schematic (older format))
At the start: 4 parts, among them U1 ARDUPROMINI, U2 RFM95

Commit message: Earth_station v1.2
Parts:
- added D1, D2: D, Diodes_ThroughHole:Diode_DO-41_SOD81_Horizontal_RM10, symbol D
- added P1: CONN_01X02, Connect:bornier2, symbol CONN_01X02
- added U3: LM2596_DC-DC, CatSat:LM2596DC-DC, symbol LM2596_DC-DC
- A1: footprint CatSat:SMA_Conn_Ant -> smd:AMPHENOL_901-144
- U1: footprint CatSat:arduinoMiniPro -> CatSat:arduinoMiniPro2
Connections:
- net GND: now also P1.1 (P1), U3.2 (IN-), U3.4 (OUT-)
- net VCC: now also D2.1 (K); no longer C1.1
- new net: D1.2 (A), P1.2 (P2)
- new net: D1.1 (K), U3.1 (IN+)
- new net (+3.3): C1.1, D2.2 (A), U3.3 (OUT+)
- no-connect marks 29 -> 23
Other:
- moved on the sheet: A1, C1, U1, U2
