File: PCB/earth_station/earth station.sch (KiCad schematic (older format))
At the start: 8 parts, among them P1 CONN_01X02, U1 ARDUPROMINI, U2 RFM95, U3 LM2596_DC-DC

Commit message: Add PDF's
Connections:
- wire segments 43 -> 46
Changed lines of the file:
@@
 EESchema Schematic File Version 2
-LIBS:earth station-rescue
 LIBS:power
 LIBS:device
@@
 LIBS:contrib
 LIBS:valves
-LIBS:rfm95
-LIBS:CatSat-cache
-LIBS:CatSat-rescue
 LIBS:earth station-cache
 EELAYER 25 0
@@
 	0    -1   -1   0
 $EndComp
-$Comp
-L GND-RESCUE-earth_station #PWR01
-U 1 1 57A11C57
-P 2280 5150
-F 0 "#PWR01" H 2280 5150 30  0001 C CNN
-F 1 "GND" H 2280 5080 30  0001 C CNN
-F 2 "" H 2280 5150 60  0000 C CNN
-F 3 "" H 2280 5150 60  0000 C CNN
-	1    2280 5150
-	1    0    0    -1
-$EndComp
-$Comp
-L GND-RESCUE-earth_station #PWR02
-U 1 1 57A11D39
-P 7020 2880
-F 0 "#PWR02" H 7020 2880 30  0001 C CNN
-F 1 "GND" H 7020 2810 30  0001 C CNN
-F 2 "" H 7020 2880 60  0000 C CNN
-F 3 "" H 7020 2880 60  0000 C CNN
-	1    7020 2880
-	1    0    0    -1
-$EndComp
 NoConn ~ 2545 4765
 NoConn ~ 2545 4865
@@
 NoConn ~ 3745 5365
 NoConn ~ 3745 5465
-$Comp
-L GND-RESCUE-earth_station #PWR03
-U 1 1 57A12CBA
-P 5620 3010
-F 0 "#PWR03" H 5620 3010 30  0001 C CNN
-F 1 "GND" H 5620 2940 30  0001 C CNN
-F 2 "" H 5620 3010 60  0000 C CNN
-F 3 "" H 5620 3010 60  0000 C CNN
-	1    5620 3010
-	1    0    0    -1
-$EndComp
-$Comp
-L GND-RESCUE-earth_station #PWR04
-U 1 1 57A12CCE
-P 5585 2285
-F 0 "#PWR04" H 5585 2285 30  0001 C CNN
-F 1 "GND" H 5585 2215 30  0001 C CNN
-F 2 "" H 5585 2285 60  0000 C CNN
-F 3 "" H 5585 2285 60  0000 C CNN
-	1    5585 2285
-	1    0    0    -1
-$EndComp
 Text Label 6925 2450 0    60   ~ 0
 INT0
 Text Label 2405 5165 0    60   ~ 0
 INT0
-$Comp
-L GND-RESCUE-earth_station #PWR05
-U 1 1 57A133C4
-P 7395 3350
-F 0 "#PWR05" H 7395 3350 30  0001 C CNN
-F 1 "GND" H 7395 3280 30  0001 C CNN
-F 2 "" H 7395 3350 60  0000 C CNN
-F 3 "" H 7395 3350 60  0000 C CNN
-	1    7395 3350
-	1    0    0    -1
-$EndComp
-$Comp
-L GND-RESCUE-earth_station #PWR06
-U 1 1 57A133F6
-P 7545 3350
-F 0 "#PWR06" H 7545 3350 30  0001 C CNN
-F 1 "GND" H 7545 3280 30  0001 C CNN
-F 2 "" H 7545 3350 60  0000 C CNN
-F 3 "" H 7545 3350 60  0000 C CNN
-	1    7545 3350
-	1    0    0    -1
-$EndComp
-$Comp
-L GND-RESCUE-earth_station #PWR07
-U 1 1 57A13487
-P 7545 2650
-F 0 "#PWR07" H 7545 2650 30  0001 C CNN
-F 1 "GND" H 7545 2580 30  0001 C CNN
-F 2 "" H 7545 2650 60  0000 C CNN
-F 3 "" H 7545 2650 60  0000 C CNN
-	1    7545 2650
-	-1   0    0    1
-$EndComp
-$Comp
-L GND-RESCUE-earth_station #PWR08
-U 1 1 57A1340A
-P 7395 2650
-F 0 "#PWR08" H 7395 2650 30  0001 C CNN
-F 1 "GND" H 7395 2580 30  0001 C CNN
-F 2 "" H 7395 2650 60  0000 C CNN
-F 3 "" H 7395 2650 60  0000 C CNN
-	1    7395 2650
-	-1   0    0    1
-$EndComp
-$Comp
-L GND-RESCUE-earth_station #PWR09
-U 1 1 57A13741
-P 5005 2860
-F 0 "#PWR09" H 5005 2860 30  0001 C CNN
-F 1 "GND" H 5005 2790 30  0001 C CNN
-F 2 "" H 5005 2860 60  0000 C CNN
-F 3 "" H 5005 2860 60  0000 C CNN
-	1    5005 2860
-	1    0    0    -1
-$EndComp
 $Comp
 L CP C1
@@
 	2280 5065 2545 5065
 Wire Wire Line
-	6830 2850 7020 2850
-Wire Wire Line
-	7020 2850 7020 2880
-Wire Wire Line
 	2280 5065 2280 5150
-Wire Wire Line
-	5585 2285 5585 2250
-Wire Wire Line
-	5585 2250 5680 2250
 Wire Wire Line
 	5620 3010 5620 2950
@@
 	1    0    0    -1
 $EndComp
-$Comp
-L GND-RESCUE-earth_station #PWR013
-U 1 1 57A677A2
-P 4170 2955
-F 0 "#PWR013" H 4170 2955 30  0001 C CNN
-F 1 "GND" H 4170 2885 30  0001 C CNN
-F 2 "" H 4170 2955 60  0000 C CNN
-F 3 "" H 4170 2955 60  0000 C CNN
-	1    4170 2955
-	1    0    0    -1
-$EndComp
 Wire Wire Line
 	4155 2690 4155 2615
@@
 Wire Wire Line
 	4170 2890 4170 2955
-$Comp
-L GND-RESCUE-earth_station #PWR014
-U 1 1 57A6805A
-P 2255 2940
-F 0 "#PWR014" H 2255 2940 30  0001 C CNN
-F 1 "GND" H 2255 2870 30  0001 C CNN
-F 2 "" H 2255 2940 60  0000 C CNN
-F 3 "" H 2255 2940 60  0000 C CNN
-	1    2255 2940
-	1    0    0    -1
-$EndComp
-$Comp
-L GND-RESCUE-earth_station #PWR015
-U 1 1 57A680EA
-P 2505 2945
-F 0 "#PWR015" H 2505 2945 30  0001 C CNN
-F 1 "GND" H 2505 2875 30  0001 C CNN
-F 2 "" H 2505 2945 60  0000 C CNN
-F 3 "" H 2505 2945 60  0000 C CNN
-	1    2505 2945
-	1    0    0    -1
-$EndComp
 $Comp
 L D D1
@@
 	1    0    0    -1
 $EndComp
+$Comp
+L GND #PWR?
+U 1 1 57C8B7E1
+P 5005 2860
+F 0 "#PWR?" H 5005 2610 50  0001 C CNN
+F 1 "GND" H 5005 2710 50  0000 C CNN
+F 2 "" H 5005 2860 50  0000 C CNN
+F 3 "" H 5005 2860 50  0000 C CNN
+	1    5005 2860
+	1    0    0    -1
+$EndComp
+$Comp
+L GND #PWR?
+U 1 1 57C8B979
+P 5620 3010
+F 0 "#PWR?" H 5620 2760 50  0001 C CNN
+F 1 "GND" H 5620 2860 50  0000 C CNN
+F 2 "" H 5620 3010 50  0000 C CNN
+F 3 "" H 5620 3010 50  0000 C CNN
+	1    5620 3010
+	1    0    0    -1
+$EndComp
+$Comp
+L GND #PWR?
+U 1 1 57C8B99C
+P 4170 2955
+F 0 "#PWR?" H 4170 2705 50  0001 C CNN
+F 1 "GND" H 4170 2805 50  0000 C CNN
+F 2 "" H 4170 2955 50  0000 C CNN
+F 3 "" H 4170 2955 50  0000 C CNN
+	1    4170 2955
+	1    0    0    -1
+$EndComp
+$Comp
+L GND #PWR?
+U 1 1 57C8BB2F
+P 2505 2945
+F 0 "#PWR?" H 2505 2695 50  0001 C CNN
+F 1 "GND" H 2505 2795 50  0000 C CNN
+F 2 "" H 2505 2945 50  0000 C CNN
+F 3 "" H 2505 2945 50  0000 C CNN
+	1    2505 2945
+	1    0    0    -1
+$EndComp
+$Comp
+L GND #PWR?
+U 1 1 57C8BC8A
+P 2255 2940
+F 0 "#PWR?" H 2255 2690 50  0001 C CNN
+F 1 "GND" H 2255 2790 50  0000 C CNN
+F 2 "" H 2255 2940 50  0000 C CNN
+F 3 "" H 2255 2940 50  0000 C CNN
+	1    2255 2940
+	1    0    0    -1
+$EndComp
+$Comp
+L GND #PWR?
+U 1 1 57C8BCAD
+P 2280 5150
+F 0 "#PWR?" H 2280 4900 50  0001 C CNN
+F 1 "GND" H 2280 5000 50  0000 C CNN
+F 2 "" H 2280 5150 50  0000 C CNN
+F 3 "" H 2280 5150 50  0000 C CNN
+	1    2280 5150
+	1    0    0    -1
+$EndComp
+$Comp
+L GND #PWR?
+U 1 1 57C8BEA0
+P 7130 2800
+F 0 "#PWR?" H 7130 2550 50  0001 C CNN
+F 1 "GND" H 7130 2650 50  0000 C CNN
+F 2 "" H 7130 2800 50  0000 C CNN
+F 3 "" H 7130 2800 50  0000 C CNN
+	1    7130 2800
+	1    0    0    -1
+$EndComp
+Wire Wire Line
+	7130 2800 7130 2780
+Wire Wire Line
+	7130 2780 6985 2780
+Wire Wire Line
+	6985 2780 6985 2850
+Wire Wire Line
+	6985 2850 6830 2850
+$Comp
+L GND #PWR?
+U 1 1 57C8C5CE
+P 5570 2175
+F 0 "#PWR?" H 5570 1925 50  0001 C CNN
+F 1 "GND" H 5570 2025 50  0000 C CNN
+F 2 "" H 5570 2175 50  0000 C CNN
+F 3 "" H 5570 2175 50  0000 C CNN
+	1    5570 2175
+	0    1    1    0
+$EndComp
+Wire Wire Line
+	5680 2250 5630 2250
+Wire Wire Line
+	5630 2250 5630 2175
+Wire Wire Line
+	5630 2175 5570 2175
+$Comp
+L GND #PWR?
+U 1 1 57C8C6EF
+P 7395 3350
+F 0 "#PWR?" H 7395 3100 50  0001 C CNN
+F 1 "GND" H 7395 3200 50  0000 C CNN
+F 2 "" H 7395 3350 50  0000 C CNN
+F 3 "" H 7395 3350 50  0000 C CNN
+	1    7395 3350
+	1    0    0    -1
+$EndComp
+$Comp
+L GND #PWR?
+U 1 1 57C8C7C2
+P 7545 3350
+F 0 "#PWR?" H 7545 3100 50  0001 C CNN
+F 1 "GND" H 7545 3200 50  0000 C CNN
+F 2 "" H 7545 3350 50  0000 C CNN
+F 3 "" H 7545 3350 50  0000 C CNN
+	1    7545 3350
+	1    0    0    -1
+$EndComp
+$Comp
+L GND #PWR?
+U 1 1 57C8C7E5
+P 7395 2650
+F 0 "#PWR?" H 7395 2400 50  0001 C CNN
+F 1 "GND" H 7395 2500 50  0000 C CNN
+F 2 "" H 7395 2650 50  0000 C CNN
+F 3 "" H 7395 2650 50  0000 C CNN
+	1    7395 2650
+	-1   0    0    1
+$EndComp
+$Comp
+L GND #PWR?
+U 1 1 57C8C8F8
+P 7545 2650
+F 0 "#PWR?" H 7545 2400 50  0001 C CNN
+F 1 "GND" H 7545 2500 50  0000 C CNN
+F 2 "" H 7545 2650 50  0000 C CNN
+F 3 "" H 7545 2650 50  0000 C CNN
+	1    7545 2650
+	-1   0    0    1
+$EndComp
 $EndSCHEMATC
