File: SensorBoard/SensorBoard.sch (KiCad schematic (older format))
At the start: 7 parts, among them P11 CONN_01X07, P12 CONN_01X04, P13 CONN_01X07, P14 CONN_01X04, P15 DHT22, P16 GY-87

Commit message: Update Schematic SensorBoard
Parts:
- C1: renamed from C2; value C -> 0.1uF
- renumbered P11 to P1, P15 to P2, P16 to P3, P12 to P4, P13 to P5, P14 to P6
Changed lines of the file:
@@
 EESchema Schematic File Version 2
-LIBS:CatSat-rescue
 LIBS:power
 LIBS:device
@@
 LIBS:contrib
 LIBS:valves
-LIBS:CatSat-cache
+LIBS:SensorBoard-cache
 EELAYER 25 0
 EELAYER END
 $Descr A4 11693 8268
 encoding utf-8
-Sheet 4 4
+Sheet 1 1
 Title "CatSat v1.0"
-Date "2016-07-26"
-Rev "0.2"
+Date "2016-10-16"
+Rev "0.3"
 Comp "Electronic Cats"
 Comment1 "Andres Sabas"
@@
 $EndDescr
 $Comp
-L CONN_01X07 P13
+L CONN_01X07 P5
 U 1 1 579A56D1
 P 7765 4620
-F 0 "P13" H 7765 5020 50  0000 C CNN
+F 0 "P5" H 7765 5020 50  0000 C CNN
 F 1 "CONN_01X07" V 7865 4620 50  0000 C CNN
 F 2 "Pin_Headers:Pin_Header_Straight_1x07" H 7765 4620 50  0001 C CNN
@@
 $EndComp
 $Comp
-L CONN_01X04 P14
+L CONN_01X04 P6
 U 1 1 579A56D8
 P 7875 3165
-F 0 "P14" H 7875 3415 50  0000 C CNN
+F 0 "P6" H 7875 3415 50  0000 C CNN
 F 1 "CONN_01X04" V 7975 3165 50  0000 C CNN
 F 2 "Pin_Headers:Pin_Header_Straight_1x04" H 7875 3165 50  0001 C CNN
@@
 Wire Wire Line
 	7190 4320 7565 4320
-Text GLabel 8570 3335 2    60   Input ~ 0
-D8
-Text GLabel 8570 3220 2    60   Input ~ 0
-D7
-Text GLabel 8570 3115 2    60   Input ~ 0
-INT1
-Text GLabel 8570 3000 2    60   Input ~ 0
-INT0
-Text GLabel 8550 4620 2    60   Input ~ 0
-MISO
-Text GLabel 8550 4505 2    60   Input ~ 0
-SCK
-Text GLabel 8550 4950 2    60   Input ~ 0
-RST
-Text GLabel 8550 4845 2    60   Input ~ 0
-NSS
-Text GLabel 8550 4730 2    60   Input ~ 0
-MOSI
-Wire Wire Line
-	8550 4505 8405 4505
-Wire Wire Line
-	8550 4620 8400 4620
-Wire Wire Line
-	8550 4730 8400 4730
-Wire Wire Line
-	8550 4845 8395 4845
-Wire Wire Line
-	8550 4950 8395 4950
-Wire Wire Line
-	8570 3000 8365 3000
-Wire Wire Line
-	8570 3115 8360 3115
-Text Label 8405 4505 2    60   ~ 0
-SCK
-Text Label 8400 4620 2    60   ~ 0
-MISO
-Text Label 8400 4730 2    60   ~ 0
-MOSI
-Text Label 8395 4845 2    60   ~ 0
-NSS
-Text Label 8395 4950 2    60   ~ 0
-RST
-Text Label 8365 3000 2    60   ~ 0
-INT0
-Text Label 8360 3115 2    60   ~ 0
-INT1
 Wire Wire Line
 	7675 3115 7520 3115
@@
 Text Label 7520 3115 0    60   ~ 0
 INT1
-Wire Wire Line
-	8360 3335 8570 3335
-Text Label 8360 3335 2    60   ~ 0
-D8
-Text Label 8365 3220 2    60   ~ 0
-D7
-Wire Wire Line
-	8365 3220 8570 3220
-$Comp
-L CONN_01X04 P12
+$Comp
+L CONN_01X04 P4
 U 1 1 579A5A85
 P 5820 2375
-F 0 "P12" H 5820 2625 50  0000 C CNN
+F 0 "P4" H 5820 2625 50  0000 C CNN
 F 1 "CONN_01X04" V 5920 2375 50  0000 C CNN
 F 2 "Pin_Headers:Pin_Header_Straight_1x04" H 5820 2375 50  0001 C CNN
@@
 $EndComp
 $Comp
-L CONN_01X07 P11
+L CONN_01X07 P1
 U 1 1 579A5A8C
 P 4520 2380
-F 0 "P11" H 4520 2780 50  0000 C CNN
+F 0 "P1" H 4520 2780 50  0000 C CNN
 F 1 "CONN_01X07" V 4620 2380 50  0000 C CNN
 F 2 "Pin_Headers:Pin_Header_Straight_1x07" H 4520 2380 50  0001 C CNN
@@
 $EndComp
 $Comp
-L +BATT #PWR027
+L +BATT #PWR01
 U 1 1 579A5A93
 P 4525 3105
-F 0 "#PWR027" H 4525 2955 50  0001 C CNN
+F 0 "#PWR01" H 4525 2955 50  0001 C CNN
 F 1 "+BATT" H 4525 3245 50  0000 C CNN
 F 2 "" H 4525 3105 50  0000 C CNN
@@
 A0
 $Comp
-L GND-RESCUE-CatSat #PWR028
+L GND-RESCUE-CatSat #PWR02
 U 1 1 579A5AA2
 P 4220 2650
-AR Path="/579A5AA2" Ref="#PWR028"  Part="1"
-AR Path="/57965E56/579A5AA2" Ref="#PWR028"  Part="1"
-F 0 "#PWR028" H 4220 2400 50  0001 C CNN
+AR Path="/579A5AA2" Ref="#PWR02"  Part="1"
+AR Path="/57965E56/579A5AA2" Ref="#PWR?"  Part="1"
+F 0 "#PWR02" H 4220 2400 50  0001 C CNN
 F 1 "GND" H 4220 2500 50  0000 C CNN
 F 2 "" H 4220 2650 50  0000 C CNN
@@
 	1    0    0    -1
 $EndComp
-Text GLabel 5985 1685 1    60   Input ~ 0
-A3
-Text GLabel 5870 1685 1    60   Input ~ 0
-A2
-Text GLabel 5765 1685 1    60   Input ~ 0
-A1
-Text GLabel 5650 1685 1    60   Input ~ 0
-A0
-Text GLabel 4545 1695 1    60   Input ~ 0
-SDA
-Text GLabel 4430 1695 1    60   Input ~ 0
-SCL
-Text GLabel 4875 1695 1    60   Input ~ 0
-DHT/D6
-Text GLabel 4770 1695 1    60   Input ~ 0
-S_TX
-Text GLabel 4655 1695 1    60   Input ~ 0
-S_RX
 Wire Wire Line
 	4620 2580 4620 2750
@@
 Wire Wire Line
 	4220 2650 4220 2580
-Wire Wire Line
-	4430 1695 4430 1840
-Wire Wire Line
-	4545 1695 4545 1845
-Wire Wire Line
-	4655 1695 4655 1845
-Wire Wire Line
-	4770 1695 4770 1850
-Wire Wire Line
-	4875 1695 4875 1850
-Wire Wire Line
-	5650 1685 5650 1890
-Wire Wire Line
-	5765 1685 5765 1895
-Wire Wire Line
-	5870 1685 5870 1890
-Wire Wire Line
-	5985 1685 5985 1895
-Text Label 4430 1840 3    60   ~ 0
-SCL
-Text Label 4545 1845 3    60   ~ 0
-SDA
-Text Label 4655 1845 3    60   ~ 0
-S_RX
-Text Label 4770 1850 3    60   ~ 0
-S_TX
-Text Label 4875 1850 3    60   ~ 0
-DHT/D6
-Text Label 5650 1890 3    60   ~ 0
-A0
-Text Label 5765 1895 3    60   ~ 0
-A1
-Text Label 5870 1890 3    60   ~ 0
-A2
-Text Label 5985 1895 3    60   ~ 0
-A3
-$Comp
-L GND-RESCUE-CatSat #PWR029
+$Comp
+L GND-RESCUE-CatSat #PWR03
 U 1 1 579A7C37
 P 7215 4505
-AR Path="/579A7C37" Ref="#PWR029"  Part="1"
-AR Path="/57965E56/579A7C37" Ref="#PWR029"  Part="1"
-F 0 "#PWR029" H 7215 4255 50  0001 C CNN
+AR Path="/579A7C37" Ref="#PWR03"  Part="1"
+AR Path="/57965E56/579A7C37" Ref="#PWR?"  Part="1"
+F 0 "#PWR03" H 7215 4255 50  0001 C CNN
 F 1 "GND" H 7215 4355 50  0000 C CNN
 F 2 "" H 7215 4505 50  0000 C CNN
@@
 $EndComp
 $Comp
-L +BATT #PWR030
+L +BATT #PWR04
 U 1 1 579A7C57
 P 7190 4250
-F 0 "#PWR030" H 7190 4100 50  0001 C CNN
+F 0 "#PWR04" H 7190 4100 50  0001 C CNN
 F 1 "+BATT" H 7190 4390 50  0000 C CNN
 F 2 "" H 7190 4250 50  0000 C CNN
@@
 	7215 4420 7215 4505
 $Comp
-L CONN_01X03 P15
+L CONN_01X03 P2
 U 1 1 579A8B76
 P 4540 4805
-F 0 "P15" H 4540 5005 50  0000 C CNN
+F 0 "P2" H 4540 5005 50  0000 C CNN
 F 1 "DHT22" V 4640 4805 50  0000 C CNN
 F 2 "Pin_Headers:Pin_Header_Straight_1x03" H 4540 4805 50  0001 C CNN
@@
 $EndComp
 $Comp
-L CONN_01X08 P16
+L CONN_01X08 P3
 U 1 1 579A8C6E
 P 5795 4855
-F 0 "P16" H 5795 5305 50  0000 C CNN
+F 0 "P3" H 5795 5305 50  0000 C CNN
 F 1 "GY-87" V 5895 4855 50  0000 C CNN
 F 2 "Pin_Headers:Pin_Header_Straight_1x08" H 5795 4855 50  0001 C CNN
@@
 SCL
 $Comp
-L +BATT #PWR031
+L +BATT #PWR05
 U 1 1 579A9426
 P 6145 4490
-F 0 "#PWR031" H 6145 4340 50  0001 C CNN
+F 0 "#PWR05" H 6145 4340 50  0001 C CNN
 F 1 "+BATT" H 6145 4630 50  0000 C CNN
 F 2 "" H 6145 4490 50  0000 C CNN
@@
 $EndComp
 $Comp
-L GND-RESCUE-CatSat #PWR032
+L GND-RESCUE-CatSat #PWR06
 U 1 1 579A9468
 P 5940 4130
-AR Path="/579A9468" Ref="#PWR032"  Part="1"
-AR Path="/57965E56/579A9468" Ref="#PWR032"  Part="1"
-F 0 "#PWR032" H 5940 3880 50  0001 C CNN
+AR Path="/579A9468" Ref="#PWR06"  Part="1"
+AR Path="/57965E56/579A9468" Ref="#PWR?"  Part="1"
+F 0 "#PWR06" H 5940 3880 50  0001 C CNN
 F 1 "GND" H 5940 3980 50  0000 C CNN
 F 2 "" H 5940 4130 50  0000 C CNN
@@
 	5940 4070 6045 4070
 $Comp
-L GND-RESCUE-CatSat #PWR033
+L GND-RESCUE-CatSat #PWR07
 U 1 1 579A95AE
 P 4280 4450
-AR Path="/579A95AE" Ref="#PWR033"  Part="1"
-AR Path="/57965E56/579A95AE" Ref="#PWR033"  Part="1"
-F 0 "#PWR033" H 4280 4200 50  0001 C CNN
+AR Path="/579A95AE" Ref="#PWR07"  Part="1"
+AR Path="/57965E56/579A95AE" Ref="#PWR?"  Part="1"
+F 0 "#PWR07" H 4280 4200 50  0001 C CNN
 F 1 "GND" H 4280 4300 50  0000 C CNN
 F 2 "" H 4280 4450 50  0000 C CNN
@@
 $EndComp
 $Comp
-L +BATT #PWR034
+L +BATT #PWR08
 U 1 1 579A95D4
 P 4540 4120
-F 0 "#PWR034" H 4540 3970 50  0001 C CNN
+F 0 "#PWR08" H 4540 3970 50  0001 C CNN
 F 1 "+BATT" H 4540 4260 50  0000 C CNN
 F 2 "" H 4540 4120 50  0000 C CNN
@@
 NoConn ~ 5645 4485
 $Comp
-L GND-RESCUE-CatSat #PWR035
+L GND-RESCUE-CatSat #PWR09
 U 1 1 579BCD75
 P 6360 4105
-AR Path="/579BCD75" Ref="#PWR035"  Part="1"
-AR Path="/57965E56/579BCD75" Ref="#PWR035"  Part="1"
-F 0 "#PWR035" H 6360 3855 50  0001 C CNN
+AR Path="/579BCD75" Ref="#PWR09"  Part="1"
+AR Path="/57965E56/579BCD75" Ref="#PWR?"  Part="1"
+F 0 "#PWR09" H 6360 3855 50  0001 C CNN
 F 1 "GND" H 6360 3955 50  0000 C CNN
 F 2 "" H 6360 4105 50  0000 C CNN
@@
 $EndComp
 $Comp
-L +BATT #PWR036
+L +BATT #PWR010
 U 1 1 579BCD92
 P 6360 3735
-F 0 "#PWR036" H 6360 3585 50  0001 C CNN
+F 0 "#PWR010" H 6360 3585 50  0001 C CNN
 F 1 "+BATT" H 6360 3875 50  0000 C CNN
 F 2 "" H 6360 3735 50  0000 C CNN
@@
 $EndComp
 $Comp
-L C C2
+L C C1
 U 1 1 579BCEC3
 P 6360 3915
-F 0 "C2" H 6385 4015 50  0000 L CNN
-F 1 "C" H 6385 3815 50  0000 L CNN
+F 0 "C1" H 6385 4015 50  0000 L CNN
+F 1 "0.1uF" H 6385 3815 50  0000 L CNN
 F 2 "Capacitors_ThroughHole:C_Disc_D6_P5" H 6398 3765 30  0001 C CNN
 F 3 "" H 6360 3915 60  0000 C CNN
@@
 $Bitmap
 Pos 9720 6850
-Scale 1.000000
+Scale 1,000000
 Data
 89 50 4E 47 0D 0A 1A 0A 00 00 00 0D 49 48 44 52 00 00 01 77 00 00 01 29 08 06 00 00 00 68 44 62
@@
 B4 9B 58 9F 89 F5 C5 4E A6 3A 93 35 43 E1 02 C8 B6 83 79 58 D3 19 67 0E 01 8E 29 B6 92 20 A6 00
 AF 03 2F 20 E9 04 FE 83 B8 0B 65 AF 55 15 F5 52 F8 7F CD 7A 0A 22 2F B5 BD D0 00 00 00 00 49 45
-4E 44 AE 42 60 82 FF
+4E 44 AE 42 60 82 00
 EndData
 $EndBitmap
