File: CommunicationBoard/CommunicationBoard.sch (KiCad schematic (older format))
At the start: 10 parts, among them P10 CONN_01X07, P7 CONN_01X07, P8 CONN_01X04, P9 CONN_01X04, U2 RFM95W-868S2

Commit message: Update Schemcatic Communication
Parts:
- C1: renamed from C3; value C -> 0.1uF
- renumbered P7 to P1, P8 to P2, P9 to P3, P10 to P4, U2 to U1
