File: GroundStation/GroundStation.kicad_pcb (KiCad board)
At the start: 2 copper layers, 57.1 x 50 mm, 13 parts, among them P1 CONN_01X02, P2 ADJ, P3 CONN_01X05, P4 CONN_01X04, U1 ARDUPROMINI, U2 RFM95, U3 LM2596_DC-DC

Commit message: Correction tracks
Routing:
- net GND: track 9.46 -> 45.5 mm, vias 4 -> 6
- net VCC: track 31.8 -> 37.0 mm
- net /INT0: track 57.6 -> 62.7 mm
Changed lines of the file:
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@@
   (general
     (links 34)
-    (no_connects 11)
-    (area 109.049999 72.599999 166.278223 122.750001)
+    (no_connects 1)
+    (area 108.972715 59.517559 178.35 123.225)
     (thickness 1.6)
     (drawings 19)
-    (tracks 127)
+    (tracks 140)
     (zones 0)
     (modules 13)
@@
   (segment (start 121.16 85.71) (end 121.2 85.75) (width 0.5) (layer B.Cu) (net 1))
   (segment (start 121.2 78.35) (end 121.16 78.31) (width 0.5) (layer B.Cu) (net 1))
+  (segment (start 144.7 110.8) (end 144.7 111.7) (width 0.3) (layer F.Cu) (net 2))
+  (segment (start 144.7 111.7) (end 144.45 111.95) (width 0.3) (layer F.Cu) (net 2))
+  (via (at 144.45 111.95) (size 0.6) (drill 0.4) (layers F.Cu B.Cu) (net 2))
+  (segment (start 141.9 108) (end 144.7 110.8) (width 0.3) (layer F.Cu) (net 2))
+  (segment (start 119.15 118.98) (end 130.13 108) (width 0.3) (layer F.Cu) (net 2))
+  (segment (start 130.13 108) (end 141.9 108) (width 0.3) (layer F.Cu) (net 2))
+  (segment (start 121.2 101.95) (end 121.2 98.5) (width 0.3) (layer B.Cu) (net 2))
+  (segment (start 121.2 98.5) (end 121.25 98.45) (width 0.3) (layer B.Cu) (net 2))
+  (via (at 121.25 98.45) (size 0.6) (drill 0.4) (layers F.Cu B.Cu) (net 2))
   (segment (start 118.12 120.03) (end 119.15 119) (width 0.3) (layer F.Cu) (net 2))
   (segment (start 119.15 119) (end 119.15 118.98) (width 0.3) (layer F.Cu) (net 2))
@@
   (segment (start 135.2 100.1) (end 135.175 100.075) (width 0.3) (layer B.Cu) (net 2))
   (via (at 135.175 100.075) (size 0.6) (drill 0.4) (layers F.Cu B.Cu) (net 2))
-  (segment (start 129.2 85.75) (end 129.2 87.25) (width 0.5) (layer B.Cu) (net 3))
-  (segment (start 117.995 104.585) (end 117.995 105.885) (width 0.5) (layer B.Cu) (net 3))
-  (segment (start 129.2 87.25) (end 117.995 98.455) (width 0.5) (layer B.Cu) (net 3))
-  (segment (start 117.995 98.455) (end 117.995 104.585) (width 0.5) (layer B.Cu) (net 3))
+  (segment (start 117.995 105.885) (end 117.995 93.205) (width 0.5) (layer B.Cu) (net 3))
+  (segment (start 117.995 93.205) (end 119.2 92) (width 0.5) (layer B.Cu) (net 3))
+  (segment (start 119.2 92) (end 128.15 92) (width 0.5) (layer B.Cu) (net 3))
+  (segment (start 128.15 92) (end 129.2 90.95) (width 0.5) (layer B.Cu) (net 3))
+  (segment (start 129.2 90.95) (end 129.2 85.75) (width 0.5) (layer B.Cu) (net 3))
   (segment (start 129.2 85.75) (end 129.2 79.45) (width 0.5) (layer B.Cu) (net 3))
   (segment (start 129.2 79.45) (end 128.7 78.95) (width 0.5) (layer B.Cu) (net 3))
+  (segment (start 141 97.55) (end 141 88.7) (width 0.3) (layer F.Cu) (net 7))
+  (segment (start 141 88.7) (end 140.5 88.2) (width 0.3) (layer F.Cu) (net 7))
+  (segment (start 140.5 88.2) (end 131.65 88.2) (width 0.3) (layer F.Cu) (net 7))
+  (segment (start 131.65 88.2) (end 131.175 87.725) (width 0.3) (layer F.Cu) (net 7))
   (segment (start 139.39 116.29) (end 140.71 116.29) (width 0.3) (layer F.Cu) (net 7))
   (segment (start 140.71 116.29) (end 141 116) (width 0.3) (layer F.Cu) (net 7))
@@
   (segment (start 131.175 85.775) (end 131.2 85.75) (width 0.3) (layer B.Cu) (net 7))
   (segment (start 141 116) (end 141 97.55) (width 0.3) (layer B.Cu) (net 7))
-  (segment (start 141 97.55) (end 131.175 87.725) (width 0.3) (layer F.Cu) (net 7))
   (via (at 131.175 87.725) (size 0.6) (drill 0.4) (layers F.Cu B.Cu) (net 7))
   (segment (start 125.2 101.95) (end 125.2 97.55) (width 0.3) (layer B.Cu) (net 9))
@@
   (segment (start 133.2 101.95) (end 133.2 105.85) (width 0.3) (layer B.Cu) (net 14))
   (segment (start 133.2 105.85) (end 133.235 105.885) (width 0.3) (layer B.Cu) (net 14))
+  (segment (start 131.2 101.95) (end 131.2 98.6) (width 0.3) (layer B.Cu) (net 15))
+  (segment (start 131.2 98.6) (end 131.775 98.025) (width 0.3) (layer B.Cu) (net 15))
+  (segment (start 131.775 98.025) (end 135.925 98.025) (width 0.3) (layer B.Cu) (net 15))
+  (segment (start 135.925 98.025) (end 136.9 99) (width 0.3) (layer B.Cu) (net 15))
+  (segment (start 136.9 99) (end 136.9 99.55521) (width 0.3) (layer B.Cu) (net 15))
   (segment (start 136.9 103.66) (end 136.9 99.55521) (width 0.3) (layer B.Cu) (net 15))
   (segment (start 136.9 99.55521) (end 136.9 99.35) (width 0.3) (layer B.Cu) (net 15))
-  (segment (start 131.2 101.95) (end 131.2 98.6) (width 0.3) (layer B.Cu) (net 15))
-  (segment (start 136.725 98.025) (end 136.9 98.2) (width 0.3) (layer B.Cu) (net 15))
-  (segment (start 131.2 98.6) (end 131.775 98.025) (width 0.3) (layer B.Cu) (net 15))
-  (segment (start 131.775 98.025) (end 136.725 98.025) (width 0.3) (layer B.Cu) (net 15))
-  (segment (start 136.9 98.2) (end 136.9 99.55521) (width 0.3) (layer B.Cu) (net 15))
   (segment (start 135.775 105.885) (end 135.775 104.785) (width 0.3) (layer B.Cu) (net 15))
   (segment (start 135.775 104.785) (end 136.9 103.66) (width 0.3) (layer B.Cu) (net 15))
