File: breakout/breakout.sch (KiCad schematic (older format))
At the start: 4 parts, among them P1 Conn_01x07_Male, P4 Conn_01x04_Male, P5 Conn_01x07_Male, P6 Conn_01x04_Male

Commit message: Update payload
Parts:
- added J1, J10, J11, J12, J13, J14, J15, J16, J17, J18, J19, J2, J20, J21, J22, J23, J24, J25, J26, J27, J28, J29, J3, J30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: D7, CatSat:Pin, symbol Connector_Generic:Conn_01x01
Connections:
- wire segments 26 -> 105
